Commit message: bittle added toe

File: bittle/urdf/bittle_toes.urdf (robot description, URDF)
Before this commit: robot bittle, 17 links, 16 joints
Links:
- link toeLB: geometry collision sphere radius=0.01; visual sphere radius=0.02
- link toeLF: geometry collision sphere radius=0.01; visual sphere radius=0.02
- link toeRB: geometry collision sphere radius=0.01; visual sphere radius=0.02
- link toeRF: geometry collision sphere radius=0.01; visual sphere radius=0.02

Commit message: bittle added toe

File: bittle/urdf/bittle_toes.urdf (robot description, URDF)
Before this commit: robot bittle, 17 links, 16 joints
Links:
- link toeLB: geometry collision sphere radius=0.01; visual sphere radius=0.05
- link toeLF: geometry collision sphere radius=0.01; visual sphere radius=0.05
- link toeRB: geometry collision sphere radius=0.01; visual sphere radius=0.05
- link toeRF: geometry collision sphere radius=0.01; visual sphere radius=0.05

Commit message: bittle added toe

File: bittle/urdf/bittle_toes.urdf (robot description, URDF)
Before this commit: robot bittle, 17 links, 16 joints
Joints:
- joint toeLB_joint: origin xyz=-0.08998 0 -0.20638 rpy=0 0 0 -> xyz=0.048254 -0.012442 -0.257702 rpy=0 0 0
- joint toeLF_joint: origin xyz=-0.09232 0 -0.20614 rpy=0 0 0 -> xyz=0.045914 -0.012442 -0.257462 rpy=0 0 0
- joint toeRB_joint: origin xyz=0.08426 -0.00238 -0.1982 rpy=0 0 0 -> xyz=0.167349 -0.016754 -0.248036 rpy=0 0 0
- joint toeRF_joint: origin xyz=0.09497 -0.00238 -0.1982 rpy=0 0 0 -> xyz=0.178059 -0.016754 -0.248036 rpy=0 0 0

Commit message: bittle added toe

File: bittle/urdf/bittle_toes.urdf (robot description, URDF)
Before this commit: robot bittle, 17 links, 16 joints
Joints:
- joint toeLB_joint: origin xyz=0.048254 -0.012442 -0.257702 rpy=0 0 0 -> xyz=-0.08998 0 -0.20638 rpy=0 0 0
- joint toeLF_joint: origin xyz=0.045914 -0.012442 -0.257462 rpy=0 0 0 -> xyz=-0.09232 0 -0.20614 rpy=0 0 0
- joint toeRB_joint: origin xyz=0.167349 -0.016754 -0.248036 rpy=0 0 0 -> xyz=0.08426 -0.00238 -0.1982 rpy=0 0 0
- joint toeRF_joint: origin xyz=0.178059 -0.016754 -0.248036 rpy=0 0 0 -> xyz=0.09497 -0.00238 -0.1982 rpy=0 0 0

Commit message: bittle added toe

File: bittle/urdf/bittle_toes.urdf (robot description, URDF)
Before this commit: robot bittle, 17 links, 16 joints
Joints:
- joint toeLF_joint: origin xyz=-0.09232 0 -0.20614 rpy=0 0 0 -> xyz=-0.9232 0 -0.20614 rpy=0 0 0

Commit message: bittle added toe

File: bittle/urdf/bittle_toes.urdf (robot description, URDF)
Before this commit: robot bittle, 17 links, 16 joints
Joints:
- joint toeLF_joint: origin xyz=-0.9232 0 -0.20614 rpy=0 0 0 -> xyz=-0.6232 0 -0.20614 rpy=0 0 0

Commit message: bittle added toe

File: bittle/urdf/bittle_toes.urdf (robot description, URDF)
Before this commit: robot bittle, 17 links, 16 joints
Joints:
- joint toeLF_joint: origin xyz=-0.6232 0 -0.20614 rpy=0 0 0 -> xyz=-0.5232 0 -0.20614 rpy=0 0 0

Commit message: bittle added toe

File: bittle/urdf/bittle_toes.urdf (robot description, URDF)
Before this commit: robot bittle, 17 links, 16 joints
Joints:
- joint toeLF_joint: origin xyz=-0.5232 0 -0.20614 rpy=0 0 0 -> xyz=-0.5 0 -0.20614 rpy=0 0 0

Commit message: bittle added toe

File: bittle/urdf/bittle_toes.urdf (robot description, URDF)
Before this commit: robot bittle, 17 links, 16 joints
Joints:
- joint toeLF_joint: origin xyz=-0.5 0 -0.20614 rpy=0 0 0 -> xyz=-0.5 0 -0.30614 rpy=0 0 0

Commit message: bittle added toe

File: bittle/urdf/bittle_toes.urdf (robot description, URDF)
Before this commit: robot bittle, 17 links, 16 joints
Joints:
- joint toeLF_joint: origin xyz=-0.5 0 -0.30614 rpy=0 0 0 -> xyz=-0.5 0 -0.1 rpy=0 0 0

Commit message: bittle added toe

File: bittle/urdf/bittle_toes.urdf (robot description, URDF)
Before this commit: robot bittle, 17 links, 16 joints
Joints:
- joint toeLB_joint: origin xyz=-0.08998 0 -0.20638 rpy=0 0 0 -> xyz=-0.5 0 -0.1 rpy=0 0 0
- joint toeRB_joint: origin xyz=0.08426 -0.00238 -0.1982 rpy=0 0 0 -> xyz=0.5 0 -0.1 rpy=0 0 0
- joint toeRF_joint: origin xyz=0.09497 -0.00238 -0.1982 rpy=0 0 0 -> xyz=0.5 0 -0.1 rpy=0 0 0
